File: catws-r2.kicad_pcb (KiCad board)
At the start: 2 copper layers, 50.1 x 50.1 mm, 88 parts, among them J1 TEST_1P, J2 TEST_1P, J3 TEST_1P, J4 TEST_1P, J5 TEST_1P, U1 ATTINY88-MU, U2 BRCC064GWZ-3

Commit message: Add missing library cache files and minor changes to firmware sensitivity thresholds
Parts:
- BT1: footprint catwsparts:CR2032-BS-6-1 -> corelib:KLS5-CR2032-11
Routing:
- net GND: track 66.4 -> 57.4 mm, vias 12 -> 13
- net Net-(D2-Pad1): track 23.5 -> 26.8 mm
- net Net-(BT1-Pad1): track 118.3 -> 121.0 mm
- net Net-(D3-Pad1): track 30.9 -> 33.2 mm
- net Net-(D4-Pad1): track 45.0 -> 46.5 mm
- net Net-(D6-Pad2): track 8.84 -> 8.23 mm
- net Net-(D6-Pad3): track 10.4 -> 9.89 mm
Other:
- board size 50.1 x 50.1 mm -> 50 x 50 mm
